Commit message: Final Version

File: urdf/arm_moveit.xacro (robot description, xacro)
@@ -2,6 +2,6 @@
 <robot name="my_arm" xmlns:xacro="http://www.ros.org/wiki/xacro">
     <xacro:include filename="$(find myroboticarm_description)/urdf/robot_parameters.xacro" />
-    <xacro:include filename="$(find myroboticarm_description)/urdf/links_joints.xacro" />
-    <!-- Virtual link to World-->
+    <xacro:include filename="$(find myroboticarm_description)/urdf/links_joints_moveit.xacro" />
+   <!-- Virtual link to World-->
     <link name="world"/>
     <joint name="world__base_link" type="fixed">

File: urdf/links_joints_moveit.xacro (robot description, xacro)
@@ -12,8 +12,8 @@
       <type>transmission_interface/SimpleTransmission</type>
       <joint name="${name}">
-        <hardwareInterface>hardware_interface/EffortJointInterface</hardwareInterface>
+        <hardwareInterface>hardware_interface/PositionJointInterface</hardwareInterface>
       </joint>
       <actuator name="motor_${name}">
-        <hardwareInterface>hardware_interface/EffortJointInterface</hardwareInterface>
+        <hardwareInterface>hardware_interface/PositionJointInterface</hardwareInterface>
         <mechanicalReduction>1</mechanicalReduction>
       </actuator>
@@ -22,4 +22,15 @@
   <xacro:macro name="m_link_cylinder" params="name origin_xyz origin_rpy radius length mass ixx ixy ixz iyy iyz izz">
     <link name="${name}">
+      <inertial>
+        <mass value="${mass}" />
+        <origin rpy="${origin_rpy}" xyz="${origin_xyz}" />
+        <inertia ixx="${ixx}" ixy="${ixy}" ixz="${ixz}" iyy="${iyy}" iyz="${iyz}" izz="${izz}" />
+      </inertial>
+      <collision>
+        <origin rpy="${origin_rpy}" xyz="${origin_xyz}" />
+        <geometry>
+          <cylinder radius="${radius}" length="${length}" />
+        </geometry>
+      </collision>
       <visual>
         <origin rpy="${origin_rpy}" xyz="${origin_xyz}" />
@@ -28,19 +39,19 @@
         </geometry>
       </visual>
-      <collision>
-        <origin rpy="${origin_rpy}" xyz="${origin_xyz}" />
-        <geometry>
-          <cylinder radius="${radius}" length="${length}" />
-        </geometry>
-        </collision>
-        <inertial>
+    </link>
+  </xacro:macro>
+  <xacro:macro name="m_link_box" params="name origin_xyz origin_rpy size mass ixx ixy ixz iyy iyz izz">
+    <link name="${name}">
+      <inertial>
         <mass value="${mass}" />
         <origin rpy="${origin_rpy}" xyz="${origin_xyz}" />
         <inertia ixx="${ixx}" ixy="${ixy}" ixz="${ixz}" iyy="${iyy}" iyz="${iyz}" izz="${izz}" />
       </inertial>
-    </link>
-  </xacro:macro>
-  <xacro:macro name="m_link_box" params="name origin_xyz origin_rpy size mass ixx ixy ixz iyy iyz izz">
-    <link name="${name}">
+      <collision>
+        <origin rpy="${origin_rpy}" xyz="${origin_xyz}" />
+        <geometry>
+          <box size="${size}" />
+        </geometry>
+      </collision>
       <visual>
         <origin rpy="${origin_rpy}" xyz="${origin_xyz}" />
@@ -49,15 +60,4 @@
         </geometry>
       </visual>
-    <collision>
-        <origin rpy="${origin_rpy}" xyz="${origin_xyz}" />
-        <geometry>
-          <box size="${size}" />
-        </geometry>
-      </collision>
-    <inertial>
-        <mass value="${mass}" />
-        <origin rpy="${origin_rpy}" xyz="${origin_xyz}" />
-        <inertia ixx="${ixx}" ixy="${ixy}" ixz="${ixz}" iyy="${iyy}" iyz="${iyz}" izz="${izz}" />
-      </inertial>
     </link>
   </xacro:macro>
